File: draft4-modular-split.brd (EAGLE design)
At the start: 100 x 88 mm, 34 parts, among them U2 SPX3819, X1 3v7 lipo, X2 ESP-12, X3 MOD-TP4056

Commit message: Pull ground back from antenna
Routing:
- net GND: track 38.3 -> 82.9 mm, vias 7 -> 6
Changed lines of the file:
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@@
 I
 G</text>
-<polygon width="1.016" layer="41">
-<vertex x="35.5" y="43.6"/>
-<vertex x="28" y="43.6"/>
-<vertex x="28" y="58.6"/>
-<vertex x="58.4" y="58.6"/>
-<vertex x="58.4" y="44"/>
-<vertex x="53" y="44"/>
-<vertex x="53" y="43.9"/>
-</polygon>
 <text x="75.8" y="22.1" size="0.8128" layer="21" ratio="18">Karl Palsson   http://false.ekta.is
 WiFi Advent rev 1 (2016)</text>
@@
 <contactref element="C31" pad="2"/>
 <contactref element="R21" pad="2"/>
-<polygon width="0.6096" layer="1" rank="2">
-<vertex x="0.5" y="72.4"/>
-<vertex x="0.5" y="0.5"/>
-<vertex x="99.5" y="0.5"/>
-<vertex x="99.5" y="72.5"/>
-<vertex x="50.1" y="87.2"/>
-<vertex x="32" y="81.9"/>
-<vertex x="30.2" y="81.2"/>
-<vertex x="27.9" y="80.5"/>
-</polygon>
 <wire x1="12.192" y1="10.8919" x2="12.192" y2="9.3" width="0.6096" layer="1"/>
 <wire x1="12.192" y1="9.3" x2="13.5" y2="9.3" width="0.6096" layer="1"/>
@@
 <wire x1="7.524" y1="68.173" x2="8.731" y2="66.9" width="0.8128" layer="1"/>
 <wire x1="8.731" y1="66.9" x2="10.1" y2="66.9" width="0.8128" layer="1"/>
-<via x="10.1" y="66.9" extent="1-16" drill="0.6"/>
 <wire x1="10.1" y1="66.9" x2="8.123" y2="66.9" width="0.8128" layer="16"/>
 <wire x1="8.123" y1="66.9" x2="7.6" y2="67.423" width="0.8128" layer="16"/>
@@
 <wire x1="90.158" y1="70.4" x2="88" y2="70.4" width="0.8128" layer="1"/>
 <via x="88" y="70.4" extent="1-16" drill="0.6"/>
-<polygon width="0.4064" layer="16">
-<vertex x="0.5" y="40"/>
-<vertex x="0.5" y="0.5"/>
-<vertex x="99.5" y="0.5"/>
-<vertex x="99.5" y="40"/>
-</polygon>
 <via x="53.6" y="26" extent="1-16" drill="0.6"/>
 <via x="55.6" y="26.5" extent="1-16" drill="0.6"/>
@@
 <contactref element="C6" pad="-"/>
 <contactref element="C7" pad="-"/>
+<wire x1="46.8" y1="77.3" x2="10.1" y2="66.9" width="1.016" layer="16" curve="-58.356796"/>
+<wire x1="7.6" y1="67.423" x2="7.6" y2="67.387121875" width="1.016" layer="16"/>
+<wire x1="7.6" y1="67.387121875" x2="3.027846875" y2="62.81496875" width="1.016" layer="16"/>
+<polygon width="0.4064" layer="16">
+<vertex x="0.6" y="0.6"/>
+<vertex x="99.5" y="0.6"/>
+<vertex x="99.5" y="72.6"/>
+<vertex x="85" y="77"/>
+<vertex x="85" y="42.9"/>
+<vertex x="25.3" y="42.9"/>
+<vertex x="14.9" y="42.9"/>
+<vertex x="14.9" y="77.1"/>
+<vertex x="0.4" y="72.7"/>
+<vertex x="0.4" y="72.2"/>
+</polygon>
+<polygon width="0.4064" layer="1">
+<vertex x="0.5" y="0.5"/>
+<vertex x="99.6" y="0.5"/>
+<vertex x="99.6" y="72.6"/>
+<vertex x="85" y="77"/>
+<vertex x="85" y="42.9"/>
+<vertex x="24.8" y="42.9"/>
+<vertex x="14.9" y="42.9"/>
+<vertex x="14.9" y="77.1"/>
+<vertex x="0.4" y="72.7"/>
+<vertex x="0.4" y="72.3"/>
+</polygon>
 </signal>
 <signal name="VBUS">
