File: hw/main-board-rev1d.sch (EAGLE design)
At the start: 34 parts, among them Q1 MOSFET-PCHANNEL, U2 MIC5504, X1 3v7 lipo, X2 ESP-12, X3 MOD-TP4056

Commit message: hw rev 1.2
Moved module to side for "proper" rf.
Fixed rotated wing connectors
Fixed overlapping polygon pours
Relaid out almost all of the lower section
Added more test points, and all spare ios on ESPmodule
Parts:
- removed C22: 10uF, microbuilder:CAP_CERAMIC0805-NOOUTLINE
- added TP1, TP2, TP3, TP4, TP5, TP6, TP7, TP8: TEST-POINTTP_06_TH, karls-parts-2016-09:TEST-POINTTP_06_TH
Connections:
- new net N$1: TP1.1, X2.GPIO16
- new net N$2: TP2.1, X2.GPIO14
- new net N$4: TP3.1, X2.GPIO12
- new net N$5: TP4.1, X2.GPIO13
- new net N$6: TP5.1, X2.GPIO5
- new net N$7: TP6.1, X2.GPIO4
- net 3.3V: no longer C22.1
- net GND: no longer C22.2
- net LEFT_IN: now also TP8.1
- net VSYS: now also TP7.1
Other:
- note added: "Solder to use diode only. (and don't populate fet diode) To use PFET, don't populate charger diode."
- note removed: "Solder to use Schottkey. never cut. no need."
- moved on the sheet: C21
Changed lines of the file:
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@@
 <part name="U$27" library="microbuilder" deviceset="GND" device=""/>
 <part name="U$28" library="microbuilder" deviceset="GND" device=""/>
-<part name="C22" library="microbuilder" deviceset="CAP_CERAMIC" device="0805-NOOUTLINE" value="10uF"/>
-<part name="U$29" library="microbuilder" deviceset="GND" device=""/>
 <part name="U$30" library="microbuilder" deviceset="GND" device=""/>
 <part name="U$3" library="microbuilder" deviceset="VBUS" device=""/>
@@
 <part name="J1" library="SparkFun-Connectors" deviceset="M04" device="1X04_NO_SILK"/>
 <part name="U$6" library="microbuilder" deviceset="3.3V" device=""/>
+<part name="TP1" library="karls-parts-2016-09" deviceset="TEST-POINT" device="TP_06_TH" value=""/>
+<part name="TP2" library="karls-parts-2016-09" deviceset="TEST-POINT" device="TP_06_TH" value=""/>
+<part name="TP3" library="karls-parts-2016-09" deviceset="TEST-POINT" device="TP_06_TH" value=""/>
+<part name="TP4" library="karls-parts-2016-09" deviceset="TEST-POINT" device="TP_06_TH" value=""/>
+<part name="TP5" library="karls-parts-2016-09" deviceset="TEST-POINT" device="TP_06_TH" value=""/>
+<part name="TP6" library="karls-parts-2016-09" deviceset="TEST-POINT" device="TP_06_TH" value=""/>
+<part name="TP7" library="karls-parts-2016-09" deviceset="TEST-POINT" device="TP_06_TH" value=""/>
+<part name="TP8" library="karls-parts-2016-09" deviceset="TEST-POINT" device="TP_06_TH" value=""/>
 </parts>
 <sheets>
@@
 . DMP3099
 . IRLML6401</text>
-<text x="50.8" y="119.38" size="1.778" layer="97">Solder to use Schottkey.
-never cut. no need.</text>
+<text x="43.18" y="116.84" size="1.778" layer="97">Solder to use diode only.
+(and don't populate fet diode)
+To use PFET, don't
+populate charger diode.</text>
 <text x="243.84" y="33.02" size="1.778" layer="97">SUCK TO MY LIBRARY AND FIX</text>
 <text x="223.52" y="15.24" size="1.778" layer="97">SUCK TO MY LIBRARY AND FIX</text>
@@
 <instances>
 <instance part="FRAME1" gate="G$3" x="134.62" y="2.54"/>
-<instance part="C21" gate="G$1" x="93.98" y="119.38"/>
+<instance part="C21" gate="G$1" x="93.98" y="114.3"/>
 <instance part="C23" gate="G$1" x="134.62" y="111.76"/>
 <instance part="U$27" gate="G$1" x="93.98" y="104.14"/>
 <instance part="U$28" gate="G$1" x="134.62" y="104.14"/>
-<instance part="C22" gate="G$1" x="127" y="111.76"/>
-<instance part="U$29" gate="G$1" x="127" y="104.14"/>
 <instance part="U$30" gate="G$1" x="104.14" y="104.14"/>
 <instance part="U$3" gate="G$1" x="12.7" y="170.18"/>
@@
 <instance part="J1" gate="G$1" x="228.6" y="55.88" rot="MR180"/>
 <instance part="U$6" gate="G$1" x="243.84" y="63.5"/>
+<instance part="TP1" gate="G$1" x="20.32" y="35.56" smashed="yes" rot="R180">
+<attribute name="NAME" x="15.24" y="35.56" size="1.778" layer="95" rot="R180"/>
+<attribute name="VALUE" x="22.86" y="38.1" size="1.778" layer="96" rot="R180"/>
+</instance>
+<instance part="TP2" gate="G$1" x="20.32" y="33.02" smashed="yes" rot="R180">
+<attribute name="NAME" x="15.24" y="33.02" size="1.778" layer="95" rot="R180"/>
+<attribute name="VALUE" x="22.86" y="35.56" size="1.778" layer="96" rot="R180"/>
+</instance>
+<instance part="TP3" gate="G$1" x="20.32" y="30.48" smashed="yes" rot="R180">
+<attribute name="NAME" x="15.24" y="30.48" size="1.778" layer="95" rot="R180"/>
+<attribute name="VALUE" x="22.86" y="33.02" size="1.778" layer="96" rot="R180"/>
+</instance>
+<instance part="TP4" gate="G$1" x="20.32" y="27.94" smashed="yes" rot="R180">
+<attribute name="NAME" x="15.24" y="27.94" size="1.778" layer="95" rot="R180"/>
+<attribute name="VALUE" x="22.86" y="30.48" size="1.778" layer="96" rot="R180"/>
+</instance>
+<instance part="TP5" gate="G$1" x="66.04" y="38.1" smashed="yes">
+<attribute name="NAME" x="71.12" y="38.1" size="1.778" layer="95"/>
+<attribute name="VALUE" x="63.5" y="35.56" size="1.778" layer="96"/>
+</instance>
+<instance part="TP6" gate="G$1" x="66.04" y="35.56" smashed="yes">
+<attribute name="NAME" x="71.12" y="35.56" size="1.778" layer="95"/>
+<attribute name="VALUE" x="63.5" y="33.02" size="1.778" layer="96"/>
+</instance>
+<instance part="TP7" gate="G$1" x="86.36" y="129.54" smashed="yes" rot="R90">
+<attribute name="NAME" x="86.36" y="134.62" size="1.778" layer="95" rot="R180"/>
+<attribute name="VALUE" x="88.9" y="127" size="1.778" layer="96" rot="R90"/>
+</instance>
+<instance part="TP8" gate="G$1" x="220.98" y="165.1" smashed="yes" rot="R90">
+<attribute name="NAME" x="218.44" y="167.64" size="1.778" layer="95" rot="R180"/>
+<attribute name="VALUE" x="223.52" y="162.56" size="1.778" layer="96" rot="R90"/>
+</instance>
 </instances>
 <busses>
@@
 <pinref part="C21" gate="G$1" pin="2"/>
 <pinref part="U$27" gate="G$1" pin="GND"/>
-<wire x1="93.98" y1="116.84" x2="93.98" y2="106.68" width="0.1524" layer="91"/>
-</segment>
-<segment>
-<pinref part="C22" gate="G$1" pin="2"/>
-<pinref part="U$29" gate="G$1" pin="GND"/>
-<wire x1="127" y1="109.22" x2="127" y2="106.68" width="0.1524" layer="91"/>
+<wire x1="93.98" y1="111.76" x2="93.98" y2="106.68" width="0.1524" layer="91"/>
 </segment>
 <segment>
@@
 </segment>
 <segment>
-<wire x1="124.46" y1="124.46" x2="127" y2="124.46" width="0.1524" layer="91"/>
-<wire x1="127" y1="124.46" x2="134.62" y2="124.46" width="0.1524" layer="91"/>
+<wire x1="124.46" y1="124.46" x2="134.62" y2="124.46" width="0.1524" layer="91"/>
 <wire x1="134.62" y1="124.46" x2="134.62" y2="127" width="0.1524" layer="91"/>
 <pinref part="C23" gate="G$1" pin="1"/>
 <wire x1="134.62" y1="124.46" x2="134.62" y2="116.84" width="0.1524" layer="91"/>
 <junction x="134.62" y="124.46"/>
-<pinref part="C22" gate="G$1" pin="1"/>
-<wire x1="127" y1="116.84" x2="127" y2="124.46" width="0.1524" layer="91"/>
-<junction x="127" y="124.46"/>
 <pinref part="U2" gate="G$1" pin="OUT"/>
 <pinref part="U$10" gate="G$1" pin="3.3V"/>
@@
 <label x="208.28" y="160.02" size="1.778" layer="95"/>
 <pinref part="R1" gate="G$1" pin="1"/>
-<wire x1="208.28" y1="160.02" x2="223.52" y2="160.02" width="0.1524" layer="91"/>
+<wire x1="208.28" y1="160.02" x2="220.98" y2="160.02" width="0.1524" layer="91"/>
+<wire x1="220.98" y1="160.02" x2="223.52" y2="160.02" width="0.1524" layer="91"/>
 <wire x1="208.28" y1="152.4" x2="208.28" y2="160.02" width="0.1524" layer="91"/>
 <pinref part="LEFT" gate="G$1" pin="2"/>
 <wire x1="208.28" y1="152.4" x2="198.12" y2="152.4" width="0.1524" layer="91"/>
+<wire x1="220.98" y1="165.1" x2="220.98" y2="160.02" width="0.1524" layer="91"/>
+<junction x="220.98" y="160.02"/>
+<pinref part="TP8" gate="G$1" pin="1"/>
 </segment>
 </net>
@@
 <wire x1="101.6" y1="121.92" x2="101.6" y2="124.46" width="0.1524" layer="91"/>
 <pinref part="C21" gate="G$1" pin="1"/>
+<wire x1="93.98" y1="119.38" x2="93.98" y2="124.46" width="0.1524" layer="91"/>
 <wire x1="93.98" y1="124.46" x2="101.6" y2="124.46" width="0.1524" layer="91"/>
 <junction x="101.6" y="124.46"/>
@@
 <label x="91.44" y="127" size="1.778" layer="95"/>
 <pinref part="JP2" gate="G$1" pin="2"/>
-<wire x1="68.58" y1="127" x2="99.06" y2="127" width="0.1524" layer="91"/>
+<wire x1="68.58" y1="127" x2="86.36" y2="127" width="0.1524" layer="91"/>
+<wire x1="86.36" y1="127" x2="99.06" y2="127" width="0.1524" layer="91"/>
+<wire x1="86.36" y1="129.54" x2="86.36" y2="127" width="0.1524" layer="91"/>
+<junction x="86.36" y="127"/>
+<pinref part="TP7" gate="G$1" pin="1"/>
 </segment>
 <segment>
@@
 </segment>
 </net>
+<net name="N$1" class="0">
+<segment>
+<pinref part="X2" gate="G$1" pin="GPIO16"/>
+<wire x1="20.32" y1="35.56" x2="25.4" y2="35.56" width="0.1524" layer="91"/>
+<pinref part="TP1" gate="G$1" pin="1"/>
+</segment>
+</net>
+<net name="N$2" class="0">
+<segment>
+<pinref part="X2" gate="G$1" pin="GPIO14"/>
+<wire x1="20.32" y1="33.02" x2="25.4" y2="33.02" width="0.1524" layer="91"/>
+<pinref part="TP2" gate="G$1" pin="1"/>
+</segment>
+</net>
+<net name="N$4" class="0">
+<segment>
+<pinref part="X2" gate="G$1" pin="GPIO12"/>
+<wire x1="20.32" y1="30.48" x2="25.4" y2="30.48" width="0.1524" layer="91"/>
+<pinref part="TP3" gate="G$1" pin="1"/>
+</segment>
+</net>
+<net name="N$5" class="0">
+<segment>
+<pinref part="X2" gate="G$1" pin="GPIO13"/>
+<wire x1="20.32" y1="27.94" x2="25.4" y2="27.94" width="0.1524" layer="91"/>
+<pinref part="TP4" gate="G$1" pin="1"/>
+</segment>
+</net>
+<net name="N$6" class="0">
+<segment>
+<pinref part="X2" gate="G$1" pin="GPIO5"/>
+<wire x1="60.96" y1="38.1" x2="66.04" y2="38.1" width="0.1524" layer="91"/>
+<pinref part="TP5" gate="G$1" pin="1"/>
+</segment>
+</net>
+<net name="N$7" class="0">
+<segment>
+<pinref part="X2" gate="G$1" pin="GPIO4"/>
+<wire x1="60.96" y1="35.56" x2="66.04" y2="35.56" width="0.1524" layer="91"/>
+<pinref part="TP6" gate="G$1" pin="1"/>
+</segment>
+</net>
